File: hw/mc unit.kicad_pcb (KiCad board)
At the start: 2 copper layers, 58 x 80 mm, 54 parts, among them J1 12 v in, J10 Conn_01x01_Female, J11 Conn_01x01_Female, J12 Conn_01x01_Female, J13 Screw_Terminal_01x12, J2 in1, J3 Screw_Terminal_01x10, J4 Conn_01x01_Female, J5 Conn_01x01_Female, J6 Conn_01x01_Female, J7 Conn_01x01_Female, J8 AVR-ISP-6, J9 Conn_01x01_Female, Q1 IRF540N, Q2 IRF540N, Q3 IRF540N, Q4 IRF540N, U1 74HC14, U2 AMS1117, U3 ATmega8L-8A, U4 ULN2003, U5 Opamp_Dual

Commit message: updated to new version of this thingamabob
Parts:
- removed the J4 at (82.5, 154.0)
- removed the R11 at (72.0, 147.0)
- removed the R12 at (72.0, 138.0)
- removed the R16 at (72.0, 126.1)
- removed the R17 at (72.0, 135.0)
- removed the U5 at (63.5, 121.5)
- added C11: C, Capacitor_SMD:C_0805_2012Metric_Pad1.18x1.45mm_HandSolder, F.Cu at (52.0, 153.5)
- added C12: C, Capacitor_SMD:C_0805_2012Metric_Pad1.18x1.45mm_HandSolder, F.Cu at (46.5, 123.0)
- added C13: C, Capacitor_SMD:C_0805_2012Metric_Pad1.18x1.45mm_HandSolder, F.Cu at (46.5, 128.0)
- added D1: LED, LED_SMD:LED_0805_2012Metric_Pad1.15x1.40mm_HandSolder, F.Cu at (48.5, 181.5)
- added D2: LED, LED_SMD:LED_0805_2012Metric_Pad1.15x1.40mm_HandSolder, F.Cu at (49.5, 153.5)
- added D3: LED, LED_SMD:LED_0805_2012Metric_Pad1.15x1.40mm_HandSolder, F.Cu at (54.5, 153.5)
- added J17: Turn Signal 1, TerminalBlock_TE-Connectivity:TerminalBlock_TE_282834-2_1x02_P2.54mm_Horizontal, F.Cu at (78.5, 118.0)
- added J18: Turn Signal 2, TerminalBlock_TE-Connectivity:TerminalBlock_TE_282834-2_1x02_P2.54mm_Horizontal, F.Cu at (78.5, 125.0)
- added J19: oil Led, TerminalBlock_TE-Connectivity:TerminalBlock_TE_282834-2_1x02_P2.54mm_Horizontal, F.Cu at (78.5, 132.0)
- added J20: Neutral Led, TerminalBlock_TE-Connectivity:TerminalBlock_TE_282834-2_1x02_P2.54mm_Horizontal, F.Cu at (78.5, 139.0)
- added J21: Turn Led, TerminalBlock_TE-Connectivity:TerminalBlock_TE_282834-2_1x02_P2.54mm_Horizontal, F.Cu at (78.5, 146.0)
- added J22: General, TerminalBlock_TE-Connectivity:TerminalBlock_TE_282834-2_1x02_P2.54mm_Horizontal, F.Cu at (78.5, 153.0)
- added J24: Conn_01x03_Male, Connector_PinHeader_2.54mm:PinHeader_1x03_P2.54mm_Vertical, F.Cu at (47.0, 110.1)
- added J26: General, TerminalBlock_TE-Connectivity:TerminalBlock_TE_282834-2_1x02_P2.54mm_Horizontal, F.Cu at (78.5, 162.3)
- added J27: General, TerminalBlock_TE-Connectivity:TerminalBlock_TE_282834-2_1x02_P2.54mm_Horizontal, F.Cu at (78.5, 169.2)
- added J28: General, TerminalBlock_TE-Connectivity:TerminalBlock_TE_282834-2_1x02_P2.54mm_Horizontal, F.Cu at (78.5, 176.1)
- added J29: General, TerminalBlock_TE-Connectivity:TerminalBlock_TE_282834-2_1x02_P2.54mm_Horizontal, F.Cu at (78.5, 183.0)
- added J8: Fuel, TerminalBlock_TE-Connectivity:TerminalBlock_TE_282834-2_1x02_P2.54mm_Horizontal, F.Cu at (34.5, 124.3)
- added R1: 6K8, Resistor_SMD:R_0603_1608Metric_Pad0.98x0.95mm_HandSolder, F.Cu at (40.5, 107.0)
- added R19: R, Resistor_SMD:R_0603_1608Metric_Pad0.98x0.95mm_HandSolder, F.Cu at (48.5, 177.5)
- added R2: 680, Resistor_SMD:R_0603_1608Metric_Pad0.98x0.95mm_HandSolder, F.Cu at (40.5, 108.5)
- added R22: 4K7, Resistor_SMD:R_0805_2012Metric_Pad1.20x1.40mm_HandSolder, F.Cu at (40.5, 158.5)
- added R23: 4K7, Resistor_SMD:R_0805_2012Metric_Pad1.20x1.40mm_HandSolder, F.Cu at (40.5, 166.0)
- added R24: 1000, Resistor_SMD:R_0805_2012Metric_Pad1.20x1.40mm_HandSolder, F.Cu at (40.5, 156.5)
- added R25: 1000, Resistor_SMD:R_0805_2012Metric_Pad1.20x1.40mm_HandSolder, F.Cu at (40.5, 164.0)
- added R26: 4K7, Resistor_SMD:R_0805_2012Metric_Pad1.20x1.40mm_HandSolder, F.Cu at (40.5, 174.0)
- added R27: 4K7, Resistor_SMD:R_0805_2012Metric_Pad1.20x1.40mm_HandSolder, F.Cu at (40.5, 182.0)
- added R28: 1000, Resistor_SMD:R_0805_2012Metric_Pad1.20x1.40mm_HandSolder, F.Cu at (40.5, 172.0)
- added R29: 1000, Resistor_SMD:R_0805_2012Metric_Pad1.20x1.40mm_HandSolder, F.Cu at (40.5, 180.0)
- added R3: 680, Resistor_SMD:R_0603_1608Metric_Pad0.98x0.95mm_HandSolder, F.Cu at (40.5, 110.0)
- added R4: 6K8, Resistor_SMD:R_0603_1608Metric_Pad0.98x0.95mm_HandSolder, F.Cu at (40.5, 115.0)
- added R5: 680, Resistor_SMD:R_0603_1608Metric_Pad0.98x0.95mm_HandSolder, F.Cu at (40.5, 116.5)
- added R6: 680, Resistor_SMD:R_0603_1608Metric_Pad0.98x0.95mm_HandSolder, F.Cu at (40.5, 118.0)
- added RV1: R_Potentiometer_Small, Potentiometer_THT:Potentiometer_Bourns_3266Y_Vertical, F.Cu at (66.9, 123.5)
- added SW1: SW_Push, Button_Switch_SMD:SW_SPST_CK_RS282G05A3, F.Cu at (66.5, 155.0)
- added U3: NCS210, Package_TO_SOT_SMD:SOT-363_SC-70-6, F.Cu at (51.5, 127.5)
- C1, C10, C2, C9: footprint Capacitor_SMD:C_1206_3216Metric -> Capacitor_SMD:C_0805_2012Metric_Pad1.18x1.45mm_HandSolder
- C3, C4, C5, C6, C8: value C -> 0,1uf; footprint Capacitor_SMD:C_1206_3216Metric -> Capacitor_SMD:C_0805_2012Metric_Pad1.18x1.45mm_HandSolder
- C7: value C -> 0.1uf; footprint Capacitor_SMD:C_1206_3216Metric -> Capacitor_SMD:C_0805_2012Metric_Pad1.18x1.45mm_HandSolder
- H1, H2: value MountingHole_4.3mm_M4 -> MountingHole; footprint MountingHole:MountingHole_4.3mm_M4 -> MountingHole:MountingHole_3.2mm_M3_DIN965
- J10: value Conn_01x01_Female -> Neutral; footprint Connector_Pin:Pin_D1.0mm_L10.0mm_LooseFit -> TerminalBlock_TE-Connectivity:TerminalBlock_TE_282834-2_1x02_P2.54mm_Horizontal
- J11: value Conn_01x01_Female -> General; footprint Connector_Pin:Pin_D1.0mm_L10.0mm_LooseFit -> TerminalBlock_TE-Connectivity:TerminalBlock_TE_282834-2_1x02_P2.54mm_Horizontal
- J16: renamed from J12; value Conn_01x01_Female -> Fuel Led; footprint Connector_Pin:Pin_D1.0mm_L10.0mm_LooseFit -> TerminalBlock_TE-Connectivity:TerminalBlock_TE_282834-2_1x02_P2.54mm_Horizontal
- J2: value in1 -> H1; footprint TerminalBlock_Phoenix:TerminalBlock_Phoenix_MPT-0,5-10-2.54_1x10_P2.54mm_Horizontal -> TerminalBlock_TE-Connectivity:TerminalBlock_TE_282834-2_1x02_P2.54mm_Horizontal
- J3: value Screw_Terminal_01x10 -> H2; footprint TerminalBlock_Phoenix:TerminalBlock_Phoenix_MPT-0,5-10-2.54_1x10_P2.54mm_Horizontal -> TerminalBlock_TE-Connectivity:TerminalBlock_TE_282834-2_1x02_P2.54mm_Horizontal
- J4: renamed from J13; value Screw_Terminal_01x12 -> H3; footprint TerminalBlock_Phoenix:TerminalBlock_Phoenix_MPT-0,5-12-2.54_1x12_P2.54mm_Horizontal -> TerminalBlock_TE-Connectivity:TerminalBlock_TE_282834-2_1x02_P2.54mm_Horizontal
- J5: value Conn_01x01_Female -> H4; footprint Connector_Pin:Pin_D1.0mm_L10.0mm_LooseFit -> TerminalBlock_TE-Connectivity:TerminalBlock_TE_282834-2_1x02_P2.54mm_Horizontal
- J6: value Conn_01x01_Female -> Blink 1; footprint Connector_Pin:Pin_D1.0mm_L10.0mm_LooseFit -> TerminalBlock_TE-Connectivity:TerminalBlock_TE_282834-2_1x02_P2.54mm_Horizontal
- J7: value Conn_01x01_Female -> Blink 2; footprint Connector_Pin:Pin_D1.0mm_L10.0mm_LooseFit -> TerminalBlock_TE-Connectivity:TerminalBlock_TE_282834-2_1x02_P2.54mm_Horizontal
- J9: value Conn_01x01_Female -> Oil; footprint Connector_Pin:Pin_D1.0mm_L10.0mm_LooseFit -> TerminalBlock_TE-Connectivity:TerminalBlock_TE_282834-2_1x02_P2.54mm_Horizontal
- Q1, Q2, Q3, Q4: value IRF540N -> AO3400A; footprint Package_TO_SOT_THT:TO-220-3_Vertical -> Package_TO_SOT_SMD:SOT-23
- R10: renamed from R4; value R -> 6K8; footprint Resistor_SMD:R_1206_3216Metric -> Resistor_SMD:R_0603_1608Metric_Pad0.98x0.95mm_HandSolder
- R11: renamed from R5; value R -> 680; footprint Resistor_SMD:R_1206_3216Metric -> Resistor_SMD:R_0603_1608Metric_Pad0.98x0.95mm_HandSolder
- R12: renamed from R6; value R -> 680; footprint Resistor_SMD:R_1206_3216Metric -> Resistor_SMD:R_0603_1608Metric_Pad0.98x0.95mm_HandSolder
- R13: value R -> 6K8; footprint Resistor_SMD:R_1206_3216Metric -> Resistor_SMD:R_0603_1608Metric_Pad0.98x0.95mm_HandSolder
- R14, R15, R18: value R -> 680; footprint Resistor_SMD:R_1206_3216Metric -> Resistor_SMD:R_0603_1608Metric_Pad0.98x0.95mm_HandSolder
- R16: renamed from R9; value R -> 6K8; footprint Resistor_SMD:R_1206_3216Metric -> Resistor_SMD:R_0603_1608Metric_Pad0.98x0.95mm_HandSolder
- R17: renamed from R10; value R -> 680; footprint Resistor_SMD:R_1206_3216Metric -> Resistor_SMD:R_0603_1608Metric_Pad0.98x0.95mm_HandSolder
- R20: renamed from R7; footprint Resistor_SMD:R_1206_3216Metric -> Resistor_SMD:R_0603_1608Metric_Pad0.98x0.95mm_HandSolder
- R21: renamed from R8; footprint Resistor_SMD:R_1206_3216Metric -> Resistor_SMD:R_0603_1608Metric_Pad0.98x0.95mm_HandSolder
- R7: renamed from R1; value R -> 6K8; footprint Resistor_SMD:R_1206_3216Metric -> Resistor_SMD:R_0603_1608Metric_Pad0.98x0.95mm_HandSolder
- R8: renamed from R2; value R -> 680; footprint Resistor_SMD:R_1206_3216Metric -> Resistor_SMD:R_0603_1608Metric_Pad0.98x0.95mm_HandSolder
- R9: renamed from R3; value R -> 680; footprint Resistor_SMD:R_1206_3216Metric -> Resistor_SMD:R_0603_1608Metric_Pad0.98x0.95mm_HandSolder
- Rshunt1, Rshunt2: footprint Resistor_SMD:R_1206_3216Metric -> Resistor_SMD:R_1206_3216Metric_Pad1.30x1.75mm_HandSolder
- U2: renamed from U1; value 74HC14 -> NCS210; footprint Package_SO:SO-14_5.3x10.2mm_P1.27mm -> Package_TO_SOT_SMD:SOT-363_SC-70-6
- U4: value ULN2003 -> ATmega8L-8A; footprint Package_SO:SOIC-16_3.9x9.9mm_P1.27mm -> Package_QFP:TQFP-32_7x7mm_P0.8mm
- U5: renamed from U3; value ATmega8L-8A -> ULN2003; footprint Package_QFP:TQFP-32_7x7mm_P0.8mm -> Package_SO:SOIC-16_3.9x9.9mm_P1.27mm
- moved J6 70.0 mm to (34.5, 108.5), turned to -90 degrees
- moved H1 68.1 mm to (65.5, 178.0)
- moved J7 60.2 mm to (34.5, 116.4), turned to -90 degrees
- moved J16 59.5 mm to (78.5, 111.0), turned to 90 degrees
- moved J9 58.1 mm to (34.5, 132.2), turned to -90 degrees
- moved J11 53.0 mm to (34.5, 148.1), turned to -90 degrees
- moved J4 52.4 mm to (34.5, 173.6), turned to -90 degrees
- moved C10 52.3 mm to (51.0, 171.0), turned to 90 degrees
- moved J5 49.6 mm to (34.5, 180.5), turned to -90 degrees
- moved J10 48.8 mm to (34.5, 140.2), turned to -90 degrees
- moved C9 48.1 mm to (62.0, 167.0), turned to -90 degrees
- moved R7 47.5 mm to (40.5, 123.0)
- moved H2 47.4 mm to (49.0, 134.0)
- moved U1 45.4 mm to (56.5, 168.5)
- moved R8 43.0 mm to (40.5, 124.5)
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- renumbered J8 to J12, U2 to U1
Connections:
- C1 pad 1: +12V -> 12 IN
- C1 pad 2: COUT -> GND
- C10 pad 1: Blink 1 ctrl -> +5V
- C10 pad 2: COUT -> GND
- C2 pad 1: Net-(C2-Pad1) -> 12 IN
- C2 pad 2: COUT -> GND
- C3 pad 2: COUT -> GND
- C4 pad 2: COUT -> GND
- C5 pad 2: COUT -> GND
- C6 pad 2: COUT -> GND
- C7 pad 2: COUT -> GND
- C8 pad 1: +5V -> Net-(C8-Pad1)
- C8 pad 2: COUT -> GND
- C9 pad 1: Blink 2 ctrl -> +5V
- C9 pad 2: COUT -> GND
- J1 pad 1: COUT -> GND
- J1 pad 2: +12V -> 12 IN
- J11 pad 1: +12V -> Net-(J11-Pad1)
- J12 pad 1: /General 1 out -> MISO
- J12 pad 3: /General 2 out -> SCK
- J12 pad 4: /Oil out -> MOSI
- J12 pad 6: COUT -> GND
- J16 pad 1: Net-(J12-Pad1) -> Fuel LEDc
- J2 pad 1: COUT -> I1
- J2 pad 2: Net-(C6-Pad1) -> 12 IN
- J3 pad 1: Net-(C7-Pad1) -> I2
- J3 pad 2: COUT -> 12 IN
- J4 pad 1: Net-(J13-Pad1) -> I3
- J4 pad 2: COUT -> 12 IN
- J5 pad 1: Net-(J5-Pad1) -> I4
- J6 pad 1: +12V -> Net-(J6-Pad1)
- J9 pad 1: +12V -> Net-(J9-Pad1)
- Q1 pad 1: i28 -> Net-(Q1-Pad1)
- Q1 pad 2: Net-(J5-Pad1) -> GND
- Q1 pad 3: COUT -> Net-(Q1-Pad3)
- Q2 pad 1: i26 -> Net-(Q2-Pad1)
- Q2 pad 2: Net-(J7-Pad1) -> GND
- Q2 pad 3: COUT -> Net-(J27-Pad1)
- Q3 pad 1: i24 -> Net-(Q3-Pad1)
- Q3 pad 2: Net-(J10-Pad1) -> GND
- Q3 pad 3: COUT -> Net-(Q3-Pad3)
- Q4 pad 1: i29 -> Net-(Q4-Pad1)
- Q4 pad 2: Net-(J12-Pad1) -> GND
- Q4 pad 3: COUT -> Net-(J29-Pad1)
- R10 pad 1: Net-(C5-Pad1) -> Net-(C6-Pad1)
- R11 pad 2: +5V -> Oil in
- R12 pad 1: Net-(C7-Pad1) -> Net-(J9-Pad1)
- R12 pad 2: +5V -> GND
- R13 pad 1: Net-(R13-Pad1) -> Net-(C7-Pad1)
- R13 pad 2: B1 Shunt -> +5V
- R14 pad 1: Net-(R14-Pad1) -> Net-(C7-Pad1)
- R14 pad 2: COUT -> Neutral in
- R15 pad 1: unconnected-(R15-Pad1) -> Net-(J10-Pad1)
- R15 pad 2: Net-(R12-Pad1) -> GND
- R16 pad 1: i24 -> Net-(C8-Pad1)
- R16 pad 2: COUT -> +5V
- R17 pad 1: i29 -> Net-(C8-Pad1)
- R17 pad 2: COUT -> General 1 in
- R18 pad 1: Net-(R18-Pad1) -> Net-(J11-Pad1)
- R18 pad 2: Blink 1 ctrl -> GND
- R20 pad 1: i28 -> Net-(R20-Pad1)
- R20 pad 2: COUT -> Net-(D2-Pad1)
- R21 pad 1: i26 -> Net-(R21-Pad1)
- R21 pad 2: COUT -> Net-(D3-Pad1)
- R7 pad 1: Net-(C2-Pad1) -> Net-(C5-Pad1)
- R8 pad 1: Net-(C3-Pad1) -> Net-(C5-Pad1)
- R8 pad 2: +5V -> fuel in
- R9 pad 1: Net-(C4-Pad1) -> Net-(J8-Pad1)
- R9 pad 2: +5V -> GND
- Rshunt1 pad 2: COUT -> Turn Sig 1c
- Rshunt2 pad 2: COUT -> Turn Sig 2c
- U1 pad 1: COUT -> GND
- U1 pad 3: +12V -> 12 IN
- U2 pad 1: Net-(C2-Pad1) -> GND
- U2 pad 2: B1 in -> GND
- U2 pad 3: Net-(C3-Pad1) -> +5V
- U2 pad 4: B2 in -> B1 Shunt
- U2 pad 5: Net-(C4-Pad1) -> Turn Sig 1c
- U2 pad 6: fuel in -> Blink 1 ctrl
- U4 pad 1: /Fuel out -> B2 in
- U4 pad 10: unconnected-(U4-Pad10) -> Neutral in
- U4 pad 11: Net-(J13-Pad11) -> General 1 in
- U4 pad 12: Net-(J13-Pad9) -> /Fuel LED out
- U4 pad 13: Net-(J13-Pad7) -> /Blink 1 out
- U4 pad 14: Net-(J13-Pad5) -> /Blink 2 out
- U4 pad 15: Net-(J13-Pad3) -> MISO
- U4 pad 16: Net-(J13-Pad1) -> MOSI
- U4 pad 2: /Blink 1 out -> Oil in
- U4 pad 3: /Blink 2 out -> GND
- U4 pad 4: /Oil out -> +5V
- U4 pad 5: /General 1 out -> GND
- U4 pad 6: /General 2 out -> +5V
- U4 pad 7: unconnected-(U4-Pad7) -> GND
- U4 pad 8: COUT -> GND
- U4 pad 9: COUT -> fuel in
- U5 pad 1: fuel in -> /Fuel LED out
- U5 pad 10: unconnected-(U3-Pad10) -> General c
- U5 pad 11: unconnected-(U3-Pad11) -> Turn Ledc
- U5 pad 12: /Fuel out -> neutral Ledc
- U5 pad 13: /Blink 1 out -> Oil Ledc
- U5 pad 14: /Blink 2 out -> Turn Sig 2c
- U5 pad 15: /Oil out -> Turn Sig 1c
- U5 pad 16: /General 1 out -> Fuel LEDc
- U5 pad 2: General 1 in -> /Blink 1 out
- U5 pad 3: COUT -> /Blink 2 out
- U5 pad 4: +5V -> /Oil out
- U5 pad 5: COUT -> /Neutral out
- U5 pad 6: +5V -> /Blink LED out
- U5 pad 7: unconnected-(U3-Pad7) -> /General 1 out
- U5 pad 8: unconnected-(U3-Pad8) -> GND
- U5 pad 9: General 2 in -> Net-(SW1-Pad1)
Routing:
- net COUT: track 438.7 -> 0.00 mm, vias 1 -> 0
- net GND: track 0.00 -> 370.5 mm, vias 0 -> 1
- net 12 IN: track 0.00 -> 182.3 mm
- net +12V: track 115.8 -> 0.00 mm, vias 2 -> 0
- net +5V: track 109.2 -> 211.3 mm, vias 1 -> 5
- net i29: track 91.6 -> 0.00 mm
- net Net-(C3-Pad1): track 89.4 -> 11.0 mm
- net Net-(C2-Pad1): track 78.4 -> 0.00 mm
- net Net-(C4-Pad1): track 71.4 -> 18.1 mm, vias 1 -> 0
- net /General 2 out: track 50.0 -> 0.00 mm, vias 2 -> 0
- net i28: track 50.0 -> 0.00 mm, vias 1 -> 0
- net MOSI: track 0.00 -> 48.3 mm, vias 0 -> 1
- net /Oil out: track 57.3 -> 12.2 mm, vias 1 -> 0
- net SCK: track 0.00 -> 43.6 mm, vias 0 -> 1
- net i24: track 43.4 -> 0.00 mm, vias 1 -> 0
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Other:
- board size 58 x 80 mm -> 53.5 x 80 mm
- board text added: "RxD"
- board text added: "TxD"

Commit message: updated to new version of this thingamabob
Parts:
- moved R22 3.50 mm to (40.5, 162.0)
- moved R24 3.50 mm to (40.5, 160.0)
- moved R23 3.00 mm to (40.5, 169.0)
- moved R25 3.00 mm to (40.5, 167.0)
- moved R26 2.00 mm to (40.5, 176.0)
- moved R28 2.00 mm to (40.5, 174.0)
- moved R27 0.48 mm to (40.5, 182.5)
- moved R29 0.48 mm to (40.5, 180.5)
Routing:
- net 12 IN: track 182.3 -> 191.8 mm, vias 0 -> 1
- net GND: track 370.5 -> 376.1 mm
- net Net-(Q1-Pad1): track 30.7 -> 29.2 mm
- net Net-(Q2-Pad1): track 30.8 -> 32.0 mm
- net Net-(Q3-Pad1): track 37.0 -> 36.1 mm
- net I2: track 7.65 -> 6.88 mm

Commit message: enhancements!
Parts:
- turned Q1 to 0 degrees
- turned Q2 to 0 degrees
- turned Q3 to 0 degrees
- turned Q4 to 0 degrees
Routing:
- net GND: track 376.1 -> 387.7 mm, vias 1 -> 4
- net Net-(Q3-Pad1): track 36.1 -> 28.9 mm, vias 0 -> 2
- net 12 IN: track 191.8 -> 196.6 mm
- net Net-(Q4-Pad1): track 29.2 -> 33.7 mm, vias 0 -> 2
- net Net-(J29-Pad1): track 10.2 -> 7.39 mm
- net Net-(Q3-Pad3): track 8.65 -> 7.33 mm
- net Net-(J27-Pad1): track 8.59 -> 7.26 mm
- net Net-(Q1-Pad3): track 8.53 -> 7.20 mm
- net Net-(Q2-Pad1): track 32.0 -> 33.0 mm, vias 0 -> 2
- net Net-(Q1-Pad1): track 29.2 -> 28.7 mm
