File: hw/mc unit.kicad_sch (KiCad schematic)
At the start: 52 parts, among them J1 12 v in, J10 Conn_01x01_Female, J11 Conn_01x01_Female, J12 Conn_01x01_Female, J13 Screw_Terminal_01x12, J2 in1, J3 Screw_Terminal_01x10, J4 Conn_01x01_Female, J5 Conn_01x01_Female, J6 Conn_01x01_Female, J7 Conn_01x01_Female, J8 AVR-ISP-6, J9 Conn_01x01_Female, Q1 IRF540N, Q2 IRF540N, Q3 IRF540N, Q4 IRF540N, U1 74HC14, U2 AMS1117, U3 ATmega8L-8A, U4 ULN2003, U5 Opamp_Dual

Commit message: updated to new version of this thingamabob
Parts:
- removed C10: C, Capacitor_SMD:C_1206_3216Metric, symbol Device:C
- removed J10, J11, J12, J4, J5, J6, J7, J9: Conn_01x01_Female, Connector_Pin:Pin_D1.0mm_L10.0mm_LooseFit, symbol Connector:Conn_01x01_Female
- removed J13: Screw_Terminal_01x12, TerminalBlock_Phoenix:TerminalBlock_Phoenix_MPT-0,5-12-2.54_1x12_P2.54mm_Horizontal, symbol Connector:Screw_Terminal_01x12
- removed J2: in1, TerminalBlock_Phoenix:TerminalBlock_Phoenix_MPT-0,5-10-2.54_1x10_P2.54mm_Horizontal, symbol Connector:Screw_Terminal_01x10
- removed J3: Screw_Terminal_01x10, TerminalBlock_Phoenix:TerminalBlock_Phoenix_MPT-0,5-10-2.54_1x10_P2.54mm_Horizontal, symbol Connector:Screw_Terminal_01x10
- removed Q1, Q2, Q3, Q4: IRF540N, Package_TO_SOT_THT:TO-220-3_Vertical, symbol Transistor_FET:IRF540N
- removed R13, R16: R, Resistor_SMD:R_1206_3216Metric, symbol Device:R
- removed U1: 74HC14, Package_SO:SO-14_5.3x10.2mm_P1.27mm, symbol 74xx:74HC14
- removed U5: Opamp_Dual, Package_SO:SOIC-8_3.9x4.9mm_P1.27mm, symbol Device:Opamp_Dual
- added C11, C12, C13, C2: C, Capacitor_SMD:C_0805_2012Metric_Pad1.18x1.45mm_HandSolder, symbol Device:C
- added D1, D2, D3: LED, LED_SMD:LED_0805_2012Metric_Pad1.15x1.40mm_HandSolder, symbol Device:LED
- added H1, H2: MountingHole, MountingHole:MountingHole_3.2mm_M3_DIN965, symbol Mechanical:MountingHole
- added J10: Neutral, TerminalBlock_TE-Connectivity:TerminalBlock_TE_282834-2_1x02_P2.54mm_Horizontal, symbol Connector:Screw_Terminal_01x02
- added J11, J22, J26, J27, J28, J29: General, TerminalBlock_TE-Connectivity:TerminalBlock_TE_282834-2_1x02_P2.54mm_Horizontal, symbol Connector:Screw_Terminal_01x02
- added J16: Fuel Led, TerminalBlock_TE-Connectivity:TerminalBlock_TE_282834-2_1x02_P2.54mm_Horizontal, symbol Connector:Screw_Terminal_01x02
- added J17: Turn Signal 1, TerminalBlock_TE-Connectivity:TerminalBlock_TE_282834-2_1x02_P2.54mm_Horizontal, symbol Connector:Screw_Terminal_01x02
- added J18: Turn Signal 2, TerminalBlock_TE-Connectivity:TerminalBlock_TE_282834-2_1x02_P2.54mm_Horizontal, symbol Connector:Screw_Terminal_01x02
- added J19: oil Led, TerminalBlock_TE-Connectivity:TerminalBlock_TE_282834-2_1x02_P2.54mm_Horizontal, symbol Connector:Screw_Terminal_01x02
- added J2: H1, TerminalBlock_TE-Connectivity:TerminalBlock_TE_282834-2_1x02_P2.54mm_Horizontal, symbol Connector:Screw_Terminal_01x02
- added J20: Neutral Led, TerminalBlock_TE-Connectivity:TerminalBlock_TE_282834-2_1x02_P2.54mm_Horizontal, symbol Connector:Screw_Terminal_01x02
- added J21: Turn Led, TerminalBlock_TE-Connectivity:TerminalBlock_TE_282834-2_1x02_P2.54mm_Horizontal, symbol Connector:Screw_Terminal_01x02
- added J24: Conn_01x03_Male, Connector_PinHeader_2.54mm:PinHeader_1x03_P2.54mm_Vertical, symbol Connector:Conn_01x03_Male
- added J3: H2, TerminalBlock_TE-Connectivity:TerminalBlock_TE_282834-2_1x02_P2.54mm_Horizontal, symbol Connector:Screw_Terminal_01x02
- added J4: H3, TerminalBlock_TE-Connectivity:TerminalBlock_TE_282834-2_1x02_P2.54mm_Horizontal, symbol Connector:Screw_Terminal_01x02
- added J5: H4, TerminalBlock_TE-Connectivity:TerminalBlock_TE_282834-2_1x02_P2.54mm_Horizontal, symbol Connector:Screw_Terminal_01x02
- added J6: Blink 1, TerminalBlock_TE-Connectivity:TerminalBlock_TE_282834-2_1x02_P2.54mm_Horizontal, symbol Connector:Screw_Terminal_01x02
- added J7: Blink 2, TerminalBlock_TE-Connectivity:TerminalBlock_TE_282834-2_1x02_P2.54mm_Horizontal, symbol Connector:Screw_Terminal_01x02
- added J8: Fuel, TerminalBlock_TE-Connectivity:TerminalBlock_TE_282834-2_1x02_P2.54mm_Horizontal, symbol Connector:Screw_Terminal_01x02
- added J9: Oil, TerminalBlock_TE-Connectivity:TerminalBlock_TE_282834-2_1x02_P2.54mm_Horizontal, symbol Connector:Screw_Terminal_01x02
- added Q1, Q2, Q3, Q4: AO3400A, Package_TO_SOT_SMD:SOT-23, symbol Transistor_FET:AO3400A
- added R19, R20, R21: R, Resistor_SMD:R_0603_1608Metric_Pad0.98x0.95mm_HandSolder, symbol Device:R
- added R2, R3, R5, R6, R8, R9: 680, Resistor_SMD:R_0603_1608Metric_Pad0.98x0.95mm_HandSolder, symbol Device:R
- added R24, R25, R28, R29: 1000, Resistor_SMD:R_0805_2012Metric_Pad1.20x1.40mm_HandSolder, symbol Device:R
- added RV1: R_Potentiometer_Small, Potentiometer_THT:Potentiometer_Bourns_3266Y_Vertical, symbol Device:R_Potentiometer_Small
- added SW1: SW_Push, Button_Switch_SMD:SW_SPST_CK_RS282G05A3, symbol Switch:SW_Push
- added U2, U3: NCS210, Package_TO_SOT_SMD:SOT-363_SC-70-6, symbol Amplifier_Current:NCS210
- C1, C9: footprint Capacitor_SMD:C_1206_3216Metric -> Capacitor_SMD:C_0805_2012Metric_Pad1.18x1.45mm_HandSolder
- C10: renamed from C8; footprint Capacitor_SMD:C_1206_3216Metric -> Capacitor_SMD:C_0805_2012Metric_Pad1.18x1.45mm_HandSolder
- C3: renamed from C2; value C -> 0,1uf; footprint Capacitor_SMD:C_1206_3216Metric -> Capacitor_SMD:C_0805_2012Metric_Pad1.18x1.45mm_HandSolder
- C4: renamed from C3; value C -> 0,1uf; footprint Capacitor_SMD:C_1206_3216Metric -> Capacitor_SMD:C_0805_2012Metric_Pad1.18x1.45mm_HandSolder
- C5: renamed from C4; value C -> 0,1uf; footprint Capacitor_SMD:C_1206_3216Metric -> Capacitor_SMD:C_0805_2012Metric_Pad1.18x1.45mm_HandSolder
- C6: renamed from C5; value C -> 0,1uf; footprint Capacitor_SMD:C_1206_3216Metric -> Capacitor_SMD:C_0805_2012Metric_Pad1.18x1.45mm_HandSolder
- C7: renamed from C6; value C -> 0.1uf; footprint Capacitor_SMD:C_1206_3216Metric -> Capacitor_SMD:C_0805_2012Metric_Pad1.18x1.45mm_HandSolder
- C8: renamed from C7; value C -> 0,1uf; footprint Capacitor_SMD:C_1206_3216Metric -> Capacitor_SMD:C_0805_2012Metric_Pad1.18x1.45mm_HandSolder
- R1: value R -> 6K8; footprint Resistor_SMD:R_1206_3216Metric -> Resistor_SMD:R_0603_1608Metric_Pad0.98x0.95mm_HandSolder
- R10: renamed from R4; value R -> 6K8; footprint Resistor_SMD:R_1206_3216Metric -> Resistor_SMD:R_0603_1608Metric_Pad0.98x0.95mm_HandSolder
- R11, R12, R14, R15, R17, R18: value R -> 680; footprint Resistor_SMD:R_1206_3216Metric -> Resistor_SMD:R_0603_1608Metric_Pad0.98x0.95mm_HandSolder
- R13: renamed from R5; value R -> 6K8; footprint Resistor_SMD:R_1206_3216Metric -> Resistor_SMD:R_0603_1608Metric_Pad0.98x0.95mm_HandSolder
- R16: renamed from R6; value R -> 6K8; footprint Resistor_SMD:R_1206_3216Metric -> Resistor_SMD:R_0603_1608Metric_Pad0.98x0.95mm_HandSolder
- R22: renamed from R9; value R -> 4K7; footprint Resistor_SMD:R_1206_3216Metric -> Resistor_SMD:R_0805_2012Metric_Pad1.20x1.40mm_HandSolder
- R23: renamed from R10; value R -> 4K7; footprint Resistor_SMD:R_1206_3216Metric -> Resistor_SMD:R_0805_2012Metric_Pad1.20x1.40mm_HandSolder
- R26: renamed from R7; value R -> 4K7; footprint Resistor_SMD:R_1206_3216Metric -> Resistor_SMD:R_0805_2012Metric_Pad1.20x1.40mm_HandSolder
- R27: renamed from R8; value R -> 4K7; footprint Resistor_SMD:R_1206_3216Metric -> Resistor_SMD:R_0805_2012Metric_Pad1.20x1.40mm_HandSolder
- R4: renamed from R2; value R -> 6K8; footprint Resistor_SMD:R_1206_3216Metric -> Resistor_SMD:R_0603_1608Metric_Pad0.98x0.95mm_HandSolder
- R7: renamed from R3; value R -> 6K8; footprint Resistor_SMD:R_1206_3216Metric -> Resistor_SMD:R_0603_1608Metric_Pad0.98x0.95mm_HandSolder
- Rshunt1, Rshunt2: footprint Resistor_SMD:R_1206_3216Metric -> Resistor_SMD:R_1206_3216Metric_Pad1.30x1.75mm_HandSolder
- renumbered J8 to J12, U2 to U1, U3 to U4, U4 to U5
Connections:
- net General 2 in is gone; now on net fuel in: U4.9 (PD5)
- net +12V: now also C2.1, J16.2 (Pin_2), J17.2 (Pin_2), J18.2 (Pin_2), J19.2 (Pin_2), J2.2 (Pin_2), J20.2 (Pin_2), J21.2 (Pin_2), J22.2 (Pin_2), J26.2 (Pin_2), J27.2 (Pin_2), J28.2 (Pin_2), J29.2 (Pin_2), J3.2 (Pin_2), J4.2 (Pin_2), J5.2 (Pin_2)
- net +5V: now also C9.1, C12.2, C13.2, D2.2 (A), D3.2 (A), R19.1, RV1.1, U2.3 (Vs), U3.3 (Vs)
- net B1 Shunt: now also J17.1 (Pin_1), U2.4 (+IN)
- net B1 in: now also U4.32 (PD2), R2.2; no longer U4.30 (PD0)
- net B2 in: now also U4.1 (PD3), R5.2; no longer U4.31 (PD1)
- net B2 shunt: now also J18.1 (Pin_1), U3.4 (+IN); no longer R11.2
- net Blink 1 ctrl: now also U4.19 (ADC6), U2.6 (OUT); no longer R18.2, U4.23 (PC0)
- net Blink 2 ctrl: now also U4.22 (ADC7), U3.6 (OUT); no longer C9.1, R17.2, U4.24 (PC1)
- net GND: now also R15.2, R18.2, U4.7 (PB6/XTAL1), U4.8 (PB7/XTAL2), C11.2, C12.1, C13.1, C2.2, D1.1 (K), J24.1 (Pin_1), Q1.2 (S), Q2.2 (S), Q3.2 (S), Q4.2 (S), R3.2, R6.2, R9.2, RV1.3, SW1.2, U2.1 (REF), U2.2 (GND), U3.1 (REF), U3.2 (GND); no longer R14.2, Rshunt1.2, Rshunt2.2, U5.9 (COM)
- net General 1 in: now also R17.2, U4.11 (PD7); no longer U4.2 (PD4)
- net General 1 out: now also U4.28 (PC5), U5.7 (I7); no longer J12.1 (MISO), U4.16 (PB4), U5.5 (I5)
- net Oil in: now also R11.2, U4.2 (PD4); no longer U4.32 (PD2)
- net Oil out: now also U4.25 (PC2); no longer J12.4 (MOSI), U4.15 (PB3)
- net fuel in: now also R8.2; no longer U4.1 (PD3)
- net at C7.1, R13.1: now also R14.1, J10.2 (Pin_2)
- net Fuel LEDc: now reaches U5.16 (O1)
- net Fuel LEDc: now also J16.1 (Pin_1)
- net Turn Ledc: now reaches U5.11 (O6)
- net Turn Ledc: now also J21.1 (Pin_1)
- net Turn Sig 1c: now reaches U5.15 (O2)
- net Turn Sig 1c: now also Rshunt1.2, U2.5 (-IN)
- net Turn Sig 2c: now reaches U5.14 (O3)
- net Turn Sig 2c: now also Rshunt2.2, U3.5 (-IN)
- net Oil Ledc: now reaches U5.13 (O4)
- net Oil Ledc: now also J19.1 (Pin_1)
- net neutral Ledc: now reaches U5.12 (O5)
- net neutral Ledc: now also J20.1 (Pin_1)
- net at R18.1: now also J11.1 (Pin_1)
- net at C6.1, R10.1: now also R11.1, J9.2 (Pin_2)
- net at C8.1, R16.1: now also R17.1, J11.2 (Pin_2)
- net at C5.1, R7.1: now also J8.2 (Pin_2), R8.1
- net at C4.1, R4.1: now also J7.2 (Pin_2), R5.1
- net at R15.1: now also J10.1 (Pin_1)
- net at R12.1: now also J9.1 (Pin_1); no longer R15.2
- net at C3.1, R1.1: now also J6.2 (Pin_2), R2.1
- net Neutral in: now reaches U4.10 (PD6)
- net Neutral in: now also R14.2
- net aref: now reaches U4.20 (AREF)
- net aref: now also C11.1, RV1.2
- net Neutral out: now reaches U4.26 (PC3)
- net Neutral out: now also U5.5 (I5)
- net Blink LED out: now reaches U4.27 (PC4)
- net Blink LED out: now also U5.6 (I6)
- net General c: now reaches U5.10 (O7)
- net General c: now also J22.1 (Pin_1)
- net Fuel out renamed Fuel LED out
- net General 2 out renamed SCK
- net SCK: no longer U5.6 (I6)
- net i24 renamed I1
- net I1: now also J2.1 (Pin_1), R24.1
- net i26 renamed I4
- net I4: now also J5.1 (Pin_1), R29.1
- net i28 renamed I3
- net I3: now also J4.1 (Pin_1), R28.1
- net i29 renamed I2
- net I2: now also J3.1 (Pin_1), R25.1
- new net: R21.1, U4.24 (PC1)
- new net: D3.1 (K), R21.2
- new net: Q1.1 (G), R24.2
- new net: J26.1 (Pin_1), Q1.3 (D)
- new net: J8.1 (Pin_1), R9.1
- new net: J28.1 (Pin_1), Q3.3 (D)
- new net: J7.1 (Pin_1), R6.1
- new net: J6.1 (Pin_1), R3.1
- new net: J27.1 (Pin_1), Q2.3 (D)
- new net: D1.2 (A), R19.2
- new net: R20.1, U4.23 (PC0)
- new net: D2.1 (K), R20.2
- new net: Q2.1 (G), R25.2
- new net: SW1.1, U5.9 (COM)
- new net: Q4.1 (G), R29.2
- new net: J29.1 (Pin_1), Q4.3 (D)
- new net: Q3.1 (G), R28.2
- new net MISO: J12.1 (MISO), U4.15 (PB3)
- new net MOSI: J12.4 (MOSI), U4.16 (PB4)
- new net RXD: J24.3 (Pin_3), U4.30 (PD0)
- new net TXD: J24.2 (Pin_2), U4.31 (PD1)
Other:
- moved on the sheet: C4, C5, C6, C7, C8, J12, R10, R13, R16, R22, R23, R26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

Commit message: enhancements!
Parts:
- C12, C13: value C -> 0.047uF
- R19, R20, R21: value R -> 100
Changed lines of the file:
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@@
   )
   (symbol (lib_id "Device:R") (at 142.24 43.18 90) (unit 1)
-    (in_bom yes) (on_board yes) (fields_autoplaced)
-    (property "Reference" "R21" (id 0) (at 142.24 38.4642 90))
-    (property "Value" "R" (id 1) (at 142.24 41.0011 90))
+    (in_bom yes) (on_board yes)
+    (property "Reference" "R21" (id 0) (at 142.24 43.18 90))
+    (property "Value" "100" (id 1) (at 142.24 45.72 90))
     (property "Footprint" "Resistor_SMD:R_0603_1608Metric_Pad0.98x0.95mm_HandSolder" (id 2) (at 142.24 44.958 90)
       (effects (font (size 1.27 1.27)) hide)
@@
     (in_bom yes) (on_board yes) (fields_autoplaced)
     (property "Reference" "C12" (id 0) (at 115.57 130.0312 90))
-    (property "Value" "C" (id 1) (at 115.57 132.5681 90))
+    (property "Value" "0.047uF" (id 1) (at 115.57 132.5681 90))
     (property "Footprint" "Capacitor_SMD:C_0805_2012Metric_Pad1.18x1.45mm_HandSolder" (id 2) (at 119.38 134.9248 0)
       (effects (font (size 1.27 1.27)) hide)
@@
   )
   (symbol (lib_id "Device:C") (at 35.56 182.88 0) (unit 1)
-    (in_bom yes) (on_board yes) (fields_autoplaced)
-    (property "Reference" "C1" (id 0) (at 38.481 182.0453 0)
-      (effects (font (size 1.27 1.27)) (justify left))
-    )
-    (property "Value" "C" (id 1) (at 38.481 184.5822 0)
+    (in_bom yes) (on_board yes)
+    (property "Reference" "C1" (id 0) (at 30.48 181.61 0)
+      (effects (font (size 1.27 1.27)) (justify left))
+    )
+    (property "Value" "C" (id 1) (at 31.75 184.15 0)
       (effects (font (size 1.27 1.27)) (justify left))
     )
@@
     (in_bom yes) (on_board yes) (fields_autoplaced)
     (property "Reference" "R19" (id 0) (at 64.77 174.3542 90))
-    (property "Value" "R" (id 1) (at 64.77 176.8911 90))
+    (property "Value" "100" (id 1) (at 64.77 176.8911 90))
     (property "Footprint" "Resistor_SMD:R_0603_1608Metric_Pad0.98x0.95mm_HandSolder" (id 2) (at 64.77 180.848 90)
       (effects (font (size 1.27 1.27)) hide)
@@
   )
   (symbol (lib_id "Device:R") (at 142.24 40.64 90) (unit 1)
-    (in_bom yes) (on_board yes) (fields_autoplaced)
-    (property "Reference" "R20" (id 0) (at 142.24 35.9242 90))
-    (property "Value" "R" (id 1) (at 142.24 38.4611 90))
+    (in_bom yes) (on_board yes)
+    (property "Reference" "R20" (id 0) (at 142.24 40.64 90))
+    (property "Value" "100" (id 1) (at 142.24 38.4611 90))
     (property "Footprint" "Resistor_SMD:R_0603_1608Metric_Pad0.98x0.95mm_HandSolder" (id 2) (at 142.24 42.418 90)
       (effects (font (size 1.27 1.27)) hide)
@@
   )
   (symbol (lib_id "Device:LED") (at 151.13 43.18 0) (unit 1)
-    (in_bom yes) (on_board yes) (fields_autoplaced)
-    (property "Reference" "D3" (id 0) (at 149.5425 38.2102 0))
-    (property "Value" "LED" (id 1) (at 149.5425 40.7471 0))
+    (in_bom yes) (on_board yes)
+    (property "Reference" "D3" (id 0) (at 153.67 41.91 0))
+    (property "Value" "LED" (id 1) (at 157.48 41.91 0))
     (property "Footprint" "LED_SMD:LED_0805_2012Metric_Pad1.15x1.40mm_HandSolder" (id 2) (at 151.13 43.18 0)
       (effects (font (size 1.27 1.27)) hide)
@@
   )
   (symbol (lib_id "Device:C") (at 40.64 182.88 0) (unit 1)
-    (in_bom yes) (on_board yes) (fields_autoplaced)
-    (property "Reference" "C2" (id 0) (at 43.561 182.0453 0)
-      (effects (font (size 1.27 1.27)) (justify left))
-    )
-    (property "Value" "C" (id 1) (at 43.561 184.5822 0)
+    (in_bom yes) (on_board yes)
+    (property "Reference" "C2" (id 0) (at 38.1 181.61 0)
+      (effects (font (size 1.27 1.27)) (justify left))
+    )
+    (property "Value" "C" (id 1) (at 38.1 185.42 0)
       (effects (font (size 1.27 1.27)) (justify left))
     )
@@
   )
   (symbol (lib_id "Device:C") (at 60.96 182.88 0) (unit 1)
-    (in_bom yes) (on_board yes) (fields_autoplaced)
-    (property "Reference" "C10" (id 0) (at 63.881 182.0453 0)
+    (in_bom yes) (on_board yes)
+    (property "Reference" "C10" (id 0) (at 63.5 181.61 0)
       (effects (font (size 1.27 1.27)) (justify left))
     )
@@
     (in_bom yes) (on_board yes) (fields_autoplaced)
     (property "Reference" "C13" (id 0) (at 115.57 161.7812 90))
-    (property "Value" "C" (id 1) (at 115.57 164.3181 90))
+    (property "Value" "0.047uF" (id 1) (at 115.57 164.3181 90))
     (property "Footprint" "Capacitor_SMD:C_0805_2012Metric_Pad1.18x1.45mm_HandSolder" (id 2) (at 119.38 166.6748 0)
       (effects (font (size 1.27 1.27)) hide)
@@
   )
   (symbol (lib_id "Device:C") (at 55.88 182.88 0) (unit 1)
-    (in_bom yes) (on_board yes) (fields_autoplaced)
-    (property "Reference" "C9" (id 0) (at 58.801 182.0453 0)
-      (effects (font (size 1.27 1.27)) (justify left))
-    )
-    (property "Value" "C" (id 1) (at 58.801 184.5822 0)
+    (in_bom yes) (on_board yes)
+    (property "Reference" "C9" (id 0) (at 53.34 180.34 0)
+      (effects (font (size 1.27 1.27)) (justify left))
+    )
+    (property "Value" "C" (id 1) (at 53.34 185.42 0)
       (effects (font (size 1.27 1.27)) (justify left))
     )
@@
   )
   (symbol (lib_id "Device:LED") (at 151.13 40.64 0) (unit 1)
-    (in_bom yes) (on_board yes) (fields_autoplaced)
-    (property "Reference" "D2" (id 0) (at 149.5425 35.6702 0))
-    (property "Value" "LED" (id 1) (at 149.5425 38.2071 0))
+    (in_bom yes) (on_board yes)
+    (property "Reference" "D2" (id 0) (at 149.86 35.56 0))
+    (property "Value" "LED" (id 1) (at 152.4 38.1 0))
     (property "Footprint" "LED_SMD:LED_0805_2012Metric_Pad1.15x1.40mm_HandSolder" (id 2) (at 151.13 40.64 0)
       (effects (font (size 1.27 1.27)) hide)
@@
     )
     (path "/2383c77e-c736-4c6a-913c-5fd14d29ae77"
-      (reference "C12") (unit 1) (value "C") (footprint "Capacitor_SMD:C_0805_2012Metric_Pad1.18x1.45mm_HandSolder")
+      (reference "C12") (unit 1) (value "0.047uF") (footprint "Capacitor_SMD:C_0805_2012Metric_Pad1.18x1.45mm_HandSolder")
     )
     (path "/e1baf61b-a25e-49b0-9d50-ee8eb67595fb"
-      (reference "C13") (unit 1) (value "C") (footprint "Capacitor_SMD:C_0805_2012Metric_Pad1.18x1.45mm_HandSolder")
+      (reference "C13") (unit 1) (value "0.047uF") (footprint "Capacitor_SMD:C_0805_2012Metric_Pad1.18x1.45mm_HandSolder")
     )
     (path "/bf9db6a1-ecac-4b06-955e-3ab661d838ec"
@@
     )
     (path "/5981cfdf-449b-45e4-80e6-4d1045a41a01"
-      (reference "R19") (unit 1) (value "R") (footprint "Resistor_SMD:R_0603_1608Metric_Pad0.98x0.95mm_HandSolder")
+      (reference "R19") (unit 1) (value "100") (footprint "Resistor_SMD:R_0603_1608Metric_Pad0.98x0.95mm_HandSolder")
     )
     (path "/59d33109-7acb-45e9-8486-3405f8d0f58b"
-      (reference "R20") (unit 1) (value "R") (footprint "Resistor_SMD:R_0603_1608Metric_Pad0.98x0.95mm_HandSolder")
+      (reference "R20") (unit 1) (value "100") (footprint "Resistor_SMD:R_0603_1608Metric_Pad0.98x0.95mm_HandSolder")
     )
     (path "/0713b836-3f2a-457f-bf5d-cebda8857401"
-      (reference "R21") (unit 1) (value "R") (footprint "Resistor_SMD:R_0603_1608Metric_Pad0.98x0.95mm_HandSolder")
+      (reference "R21") (unit 1) (value "100") (footprint "Resistor_SMD:R_0603_1608Metric_Pad0.98x0.95mm_HandSolder")
     )
     (path "/7640d122-a1c8-4633-ad07-0b7de59186d0"
